File: v1/9902_taipo.brd (EAGLE design)
At the start: 10 x 106 mm, 22 parts, among them IC1 1117-5.0, IC4 1117-3.3, J10 PJ301CM, J11 PJ301CM, J21 EURO_POWER_LOCK, U1 74LV1T34SOT23-5, U2 TLP2366(V4-TPL,E

Commit message: Resized for JLCPCB price optimisation
Other:
- board size 10 x 106 mm -> 10 x 99 mm
Changed lines of the file:
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@@
 <board>
 <plain>
-<wire x1="0" y1="0" x2="10" y2="0" width="0" layer="20"/>
-<wire x1="10" y1="0" x2="10" y2="105.95" width="0" layer="20"/>
+<wire x1="0" y1="7" x2="10" y2="7" width="0" layer="20"/>
+<wire x1="10" y1="7" x2="10" y2="105.95" width="0" layer="20"/>
 <wire x1="10" y1="105.95" x2="0" y2="105.95" width="0" layer="20"/>
-<wire x1="0" y1="105.95" x2="0" y2="0" width="0" layer="20"/>
+<wire x1="0" y1="105.95" x2="0" y2="7" width="0" layer="20"/>
 <text x="1.66" y="78.585" size="0.8" layer="21" font="vector" ratio="14" rot="R90"> JLCJLCJLCJLC</text>
 </plain>
@@
 <vertex x="0" y="106.045"/>
 <vertex x="10" y="106.045"/>
-<vertex x="10" y="0"/>
-<vertex x="0" y="0"/>
+<vertex x="10" y="7.05"/>
+<vertex x="0" y="7.05"/>
 </polygon>
 <polygon width="0.1524" layer="16">
 <vertex x="0" y="106.045"/>
 <vertex x="9.905" y="106.045"/>
-<vertex x="9.905" y="0"/>
-<vertex x="0" y="0"/>
+<vertex x="9.905" y="7.15"/>
+<vertex x="0" y="7.15"/>
 </polygon>
 <contactref element="U1" pad="3"/>
